File: SchmaticAndPcb/TurnLightSignalAssistance/TurnLightSignalAssistance.kicad_pcb (KiCad board)
At the start: 2 copper layers, 3 parts, among them J1 SSD1306_LCD, J2 MPU6050

Commit message: fixing and optimizing schematic
Parts:
- removed J1: SSD1306_LCD, Connector_PinSocket_2.54mm:PinSocket_1x04_P2.54mm_Vertical
- added D1: LED, LED_THT:LED_D3.0mm, F.Cu at (161.8, 79.8)
- added D2: LED, LED_THT:LED_D3.0mm, F.Cu at (182.2, 59.9)
- added D3: LED, LED_THT:LED_D3.0mm, F.Cu at (172.7, 68.3)
- added D4: LED, LED_THT:LED_D3.0mm, F.Cu at (178.6, 68.3)
- added D5: LED, LED_THT:LED_D3.0mm, F.Cu at (167.7, 79.8)
- added D6: LED, LED_THT:LED_D3.0mm, F.Cu at (161.8, 85.3)
- added D9: LED, LED_THT:LED_D3.0mm, F.Cu at (188.8, 54.1)
- added Q1: 2SC1815, Package_TO_SOT_THT:TO-92_Inline, F.Cu at (182.6, 54.5)
- added R1: 1K, Resistor_THT:R_Axial_DIN0309_L9.0mm_D3.2mm_P12.70mm_Horizontal, F.Cu at (142.4, 100.9)
- added R10: 1K, Resistor_THT:R_Axial_DIN0309_L9.0mm_D3.2mm_P12.70mm_Horizontal, F.Cu at (126.5, 100.9)
- added R11: 10K, Resistor_THT:R_Axial_DIN0309_L9.0mm_D3.2mm_P12.70mm_Horizontal, F.Cu at (145.8, 80.8)
- added R12: 220, Resistor_THT:R_Axial_DIN0309_L9.0mm_D3.2mm_P12.70mm_Horizontal, F.Cu at (166.3, 58.4)
- added R2: 1K, Resistor_THT:R_Axial_DIN0309_L9.0mm_D3.2mm_P12.70mm_Horizontal, F.Cu at (150.4, 53.7)
- added R3: 1K, Resistor_THT:R_Axial_DIN0309_L9.0mm_D3.2mm_P12.70mm_Horizontal, F.Cu at (150.4, 63.2)
- added R4: 1K, Resistor_THT:R_Axial_DIN0309_L9.0mm_D3.2mm_P12.70mm_Horizontal, F.Cu at (166.3, 53.7)
- added R5: 1K, Resistor_THT:R_Axial_DIN0309_L9.0mm_D3.2mm_P12.70mm_Horizontal, F.Cu at (145.8, 76.1)
- added R6: 1K, Resistor_THT:R_Axial_DIN0309_L9.0mm_D3.2mm_P12.70mm_Horizontal, F.Cu at (150.4, 67.9)
- added R7: 1K, Resistor_THT:R_Axial_DIN0309_L9.0mm_D3.2mm_P12.70mm_Horizontal, F.Cu at (150.4, 58.4)
- added R8: 1K, Resistor_THT:R_Axial_DIN0309_L9.0mm_D3.2mm_P12.70mm_Horizontal, F.Cu at (145.8, 85.6)
- added R9: 1K, Resistor_THT:R_Axial_DIN0309_L9.0mm_D3.2mm_P12.70mm_Horizontal, F.Cu at (166.3, 63.2)
- added U2: PC817, Package_DIP:DIP-4_W7.62mm, F.Cu at (161.8, 72.4)
- added U3: PC817, Package_DIP:DIP-4_W7.62mm, F.Cu at (145.9, 90.0)
- moved J2 61.9 mm to (146.6, 53.6)
- moved A1 20.5 mm to (127.0, 55.9)
Connections:
- A1 pad 12: /EnableFunction -> /AliveLed
- A1 pad 13: /BlinkLeft -> /SignalRight
- A1 pad 14: /BlinkRight -> /SignalLeft
- A1 pad 15: /SignalLeft -> /LightControl
- A1 pad 16: /SignalRight -> unconnected-(A1-Pad16)
- A1 pad 27: unconnected-(A1-Pad27) -> Net-(A1-Pad27)
- A1 pad 30: VCC -> unconnected-(A1-Pad30)
- J2 pad 1: VCC -> +5V
